File: Final_project_rbree/Final_project_rbree.kicad_sch (KiCad schematic)
At the start: 44 parts, among them J1 Conn_01x02_Pin, J2 Conn_01x02_Pin, Q1 MMBT3904, Q2 AO3401A, U1 TL431, U2 LTV-817, U3 B1212, U4 2N7002, U7 NE555

Commit message: Add files via upload
Parts:
- added H1, H2, H3, H4: MountingHole, MountingHole:MountingHole_3.2mm_M3, symbol Mechanical:MountingHole

Commit message: Add files via upload
Parts:
- H1, H2, H3, H4: footprint MountingHole:MountingHole_3.2mm_M3 -> MountingHole:MountingHole_3mm
Other:
- moved on the sheet: H1, H2, H3, H4
Changed lines of the file:
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@@
 	(symbol
 		(lib_id "Mechanical:MountingHole")
-		(at 135.89 249.555 0)
+		(at 130.175 201.93 0)
 		(unit 1)
 		(exclude_from_sim yes)
@@
 		(fields_autoplaced yes)
 		(property "Reference" "H1"
-			(at 138.43 248.2849 0)
+			(at 132.715 200.6599 0)
 			(effects
 				(font
@@
 		)
 		(property "Value" "MountingHole"
-			(at 138.43 250.8249 0)
-			(effects
-				(font
-					(size 1.27 1.27)
-				)
-				(justify left)
-			)
-		)
-		(property "Footprint" "MountingHole:MountingHole_3.2mm_M3"
-			(at 135.89 249.555 0)
+			(at 132.715 203.1999 0)
+			(effects
+				(font
+					(size 1.27 1.27)
+				)
+				(justify left)
+			)
+		)
+		(property "Footprint" "MountingHole:MountingHole_3mm"
+			(at 130.175 201.93 0)
 			(effects
 				(font
@@
 		)
 		(property "Datasheet" "~"
-			(at 135.89 249.555 0)
+			(at 130.175 201.93 0)
 			(effects
 				(font
@@
 		)
 		(property "Description" "Mounting Hole without connection"
-			(at 135.89 249.555 0)
+			(at 130.175 201.93 0)
 			(effects
 				(font
@@
 	(symbol
 		(lib_id "power:VCC")
-		(at 152.4 38.1 180)
+		(at 160.655 85.09 180)
 		(unit 1)
 		(exclude_from_sim no)
@@
 		(dnp no)
 		(property "Reference" "#PWR023"
-			(at 152.4 34.29 0)
+			(at 160.655 81.28 0)
 			(effects
 				(font
@@
 		)
 		(property "Value" "VCC"
-			(at 151.9682 42.4942 0)
+			(at 160.2232 89.4842 0)
 			(effects
 				(font
@@
 		)
 		(property "Footprint" ""
-			(at 152.4 38.1 0)
+			(at 160.655 85.09 0)
 			(effects
 				(font
@@
 		)
 		(property "Datasheet" ""
-			(at 152.4 38.1 0)
+			(at 160.655 85.09 0)
 			(effects
 				(font
@@
 		)
 		(property "Description" ""
-			(at 152.4 38.1 0)
+			(at 160.655 85.09 0)
 			(effects
 				(font
@@
 	(symbol
 		(lib_id "power:PWR_FLAG")
-		(at 146.05 38.1 0)
+		(at 154.305 85.09 0)
 		(unit 1)
 		(exclude_from_sim no)
@@
 		(fields_autoplaced yes)
 		(property "Reference" "#FLG01"
-			(at 146.05 36.195 0)
+			(at 154.305 83.185 0)
 			(effects
 				(font
@@
 		)
 		(property "Value" "PWR_FLAG"
-			(at 146.05 33.655 0)
+			(at 154.305 80.645 0)
 			(effects
 				(font
@@
 		)
 		(property "Footprint" ""
-			(at 146.05 38.1 0)
+			(at 154.305 85.09 0)
 			(effects
 				(font
@@
 		)
 		(property "Datasheet" "~"
-			(at 146.05 38.1 0)
+			(at 154.305 85.09 0)
 			(effects
 				(font
@@
 		)
 		(property "Description" "Special symbol for telling ERC where power comes from"
-			(at 146.05 38.1 0)
+			(at 154.305 85.09 0)
 			(effects
 				(font
@@
 	(symbol
 		(lib_id "power:PWR_FLAG")
-		(at 139.7 38.1 0)
+		(at 147.955 85.09 0)
 		(unit 1)
 		(exclude_from_sim no)
@@
 		(fields_autoplaced yes)
 		(property "Reference" "#FLG03"
-			(at 139.7 36.195 0)
+			(at 147.955 83.185 0)
 			(effects
 				(font
@@
 		)
 		(property "Value" "PWR_FLAG"
-			(at 139.7 33.655 0)
+			(at 147.955 80.645 0)
 			(effects
 				(font
@@
 		)
 		(property "Footprint" ""
-			(at 139.7 38.1 0)
+			(at 147.955 85.09 0)
 			(effects
 				(font
@@
 		)
 		(property "Datasheet" "~"
-			(at 139.7 38.1 0)
+			(at 147.955 85.09 0)
 			(effects
 				(font
@@
 		)
 		(property "Description" "Special symbol for telling ERC where power comes from"
-			(at 139.7 38.1 0)
+			(at 147.955 85.09 0)
 			(effects
 				(font
@@
 	(symbol
 		(lib_id "power:PWR_FLAG")
-		(at 152.4 38.1 0)
+		(at 160.655 85.09 0)
 		(unit 1)
 		(exclude_from_sim no)
@@
 		(fields_autoplaced yes)
 		(property "Reference" "#FLG02"
-			(at 152.4 36.195 0)
+			(at 160.655 83.185 0)
 			(effects
 				(font
@@
 		)
 		(property "Value" "PWR_FLAG"
-			(at 152.4 33.655 0)
+			(at 160.655 80.645 0)
 			(effects
 				(font
@@
 		)
 		(property "Footprint" ""
-			(at 152.4 38.1 0)
+			(at 160.655 85.09 0)
 			(effects
 				(font
@@
 		)
 		(property "Datasheet" "~"
-			(at 152.4 38.1 0)
+			(at 160.655 85.09 0)
 			(effects
 				(font
@@
 		)
 		(property "Description" "Special symbol for telling ERC where power comes from"
-			(at 152.4 38.1 0)
+			(at 160.655 85.09 0)
 			(effects
 				(font
@@
 	(symbol
 		(lib_id "Mechanical:MountingHole")
-		(at 135.89 266.065 0)
+		(at 130.175 218.44 0)
 		(unit 1)
 		(exclude_from_sim yes)
@@
 		(fields_autoplaced yes)
 		(property "Reference" "H4"
-			(at 138.43 264.7949 0)
+			(at 132.715 217.1699 0)
 			(effects
 				(font
@@
 		)
 		(property "Value" "MountingHole"
-			(at 138.43 267.3349 0)
-			(effects
-				(font
-					(size 1.27 1.27)
-				)
-				(justify left)
-			)
-		)
-		(property "Footprint" "MountingHole:MountingHole_3.2mm_M3"
-			(at 135.89 266.065 0)
+			(at 132.715 219.7099 0)
+			(effects
+				(font
+					(size 1.27 1.27)
+				)
+				(justify left)
+			)
+		)
+		(property "Footprint" "MountingHole:MountingHole_3mm"
+			(at 130.175 218.44 0)
 			(effects
 				(font
@@
 		)
 		(property "Datasheet" "~"
-			(at 135.89 266.065 0)
+			(at 130.175 218.44 0)
 			(effects
 				(font
@@
 		)
 		(property "Description" "Mounting Hole without connection"
-			(at 135.89 266.065 0)
+			(at 130.175 218.44 0)
 			(effects
 				(font
@@
 	(symbol
 		(lib_id "power-symbol-library:GLV+")
-		(at 146.05 38.1 0)
+		(at 154.305 85.09 0)
 		(mirror x)
 		(unit 1)
@@
 		(dnp no)
 		(property "Reference" "#PWR022"
-			(at 146.05 34.29 0)
+			(at 154.305 81.28 0)
 			(effects
 				(font
@@
 		)
 		(property "Value" "GLV+"
-			(at 146.431 42.4942 0)
+			(at 154.686 89.4842 0)
 			(effects
 				(font
@@
 		)
 		(property "Footprint" ""
-			(at 146.05 38.1 0)
+			(at 154.305 85.09 0)
 			(effects
 				(font
@@
 		)
 		(property "Datasheet" ""
-			(at 146.05 38.1 0)
+			(at 154.305 85.09 0)
 			(effects
 				(font
@@
 		)
 		(property "Description" ""
-			(at 146.05 38.1 0)
+			(at 154.305 85.09 0)
 			(effects
 				(font
@@
 	(symbol
 		(lib_id "power-symbol-library:GLV+")
-		(at 139.7 38.1 0)
+		(at 147.955 85.09 0)
 		(mirror x)
 		(unit 1)
@@
 		(dnp no)
 		(property "Reference" "#PWR024"
-			(at 139.7 34.29 0)
+			(at 147.955 81.28 0)
 			(effects
 				(font
@@
 		)
 		(property "Value" "GLV-"
-			(at 140.081 42.4942 0)
+			(at 148.336 89.4842 0)
 			(effects
 				(font
@@
 		)
 		(property "Footprint" ""
-			(at 139.7 38.1 0)
+			(at 147.955 85.09 0)
 			(effects
 				(font
@@
 		)
 		(property "Datasheet" ""
-			(at 139.7 38.1 0)
+			(at 147.955 85.09 0)
 			(effects
 				(font
@@
 		)
 		(property "Description" ""
-			(at 139.7 38.1 0)
+			(at 147.955 85.09 0)
 			(effects
 				(font
@@
 	(symbol
 		(lib_id "Mechanical:MountingHole")
-		(at 135.89 254.635 0)
+		(at 130.175 207.01 0)
 		(unit 1)
 		(exclude_from_sim yes)
@@
 		(fields_autoplaced yes)
 		(property "Reference" "H2"
-			(at 138.43 253.3649 0)
+			(at 132.715 205.7399 0)
 			(effects
 				(font
@@
 		)
 		(property "Value" "MountingHole"
-			(at 138.43 255.9049 0)
-			(effects
-				(font
-					(size 1.27 1.27)
-				)
-				(justify left)
-			)
-		)
-		(property "Footprint" "MountingHole:MountingHole_3.2mm_M3"
-			(at 135.89 254.635 0)
+			(at 132.715 208.2799 0)
+			(effects
+				(font
+					(size 1.27 1.27)
+				)
+				(justify left)
+			)
+		)
+		(property "Footprint" "MountingHole:MountingHole_3mm"
+			(at 130.175 207.01 0)
 			(effects
 				(font
@@
 		)
 		(property "Datasheet" "~"
-			(at 135.89 254.635 0)
+			(at 130.175 207.01 0)
 			(effects
 				(font
@@
 		)
 		(property "Description" "Mounting Hole without connection"
-			(at 135.89 254.635 0)
+			(at 130.175 207.01 0)
 			(effects
 				(font
@@
 	(symbol
 		(lib_id "Mechanical:MountingHole")
-		(at 135.89 260.35 0)
+		(at 130.175 212.725 0)
 		(unit 1)
 		(exclude_from_sim yes)
@@
 		(fields_autoplaced yes)
 		(property "Reference" "H3"
-			(at 138.43 259.0799 0)
+			(at 132.715 211.4549 0)
 			(effects
 				(font
@@
 		)
 		(property "Value" "MountingHole"
-			(at 138.43 261.6199 0)
-			(effects
-				(font
-					(size 1.27 1.27)
-				)
-				(justify left)
-			)
-		)
-		(property "Footprint" "MountingHole:MountingHole_3.2mm_M3"
-			(at 135.89 260.35 0)
+			(at 132.715 213.9949 0)
+			(effects
+				(font
+					(size 1.27 1.27)
+				)
+				(justify left)
+			)
+		)
+		(property "Footprint" "MountingHole:MountingHole_3mm"
+			(at 130.175 212.725 0)
 			(effects
 				(font
@@
 		)
 		(property "Datasheet" "~"
-			(at 135.89 260.35 0)
+			(at 130.175 212.725 0)
 			(effects
 				(font
@@
 		)
 		(property "Description" "Mounting Hole without connection"
-			(at 135.89 260.35 0)
-			(effects
-				(font
+			(at 130.175 212.725 0)
+			(effects
+				(font

Commit message: Add files via upload
Parts:
- H1, H2, H3, H4: footprint MountingHole:MountingHole_3mm -> MountingHole:MountingHole_3.2mm_M3
Changed lines of the file:
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@@
 			)
 		)
-		(property "Footprint" "MountingHole:MountingHole_3mm"
+		(property "Footprint" "MountingHole:MountingHole_3.2mm_M3"
 			(at 130.175 201.93 0)
 			(effects
@@
 			)
 		)
-		(property "Footprint" "MountingHole:MountingHole_3mm"
+		(property "Footprint" "MountingHole:MountingHole_3.2mm_M3"
 			(at 130.175 218.44 0)
 			(effects
@@
 			)
 		)
-		(property "Footprint" "MountingHole:MountingHole_3mm"
+		(property "Footprint" "MountingHole:MountingHole_3.2mm_M3"
 			(at 130.175 207.01 0)
 			(effects
@@
 			)
 		)
-		(property "Footprint" "MountingHole:MountingHole_3mm"
+		(property "Footprint" "MountingHole:MountingHole_3.2mm_M3"
 			(at 130.175 212.725 0)
 			(effects
